Commit message: modified urdf, env cfg

File: source/M20_Piper/M20_Piper/assets/M20_Piper.urdf (robot description, URDF)
Before this commit: robot M20_Piper, 27 links, 26 joints
Links:
- added link front_lidar; visual box size=0.05 0.05 0.04
Joints:
- added joint base_to_front_lidar: type fixed, parent base_link, child front_lidar, origin xyz=0.37 0.0 0.05 rpy=0 0.12 0
