Commit message: stage 1. path tracking without obstacle

File: source/M20_Piper/M20_Piper/assets/M20_Piper.urdf (robot description, URDF)
Before this commit: robot M20_Piper, 28 links, 27 joints
Joints:
- joint fl_hipx_joint: axis -1 0 0 -> (none); limit lower=-0.611 upper=0.436 effort=76.4 velocity=22.4 -> (none); type revolute -> fixed
- joint fl_hipy_joint: axis 0 -1 0 -> (none); limit lower=-2.583 upper=2.286 effort=76.4 velocity=22.4 -> (none); origin xyz=0 0 0 rpy=0 0 0 -> xyz=0 0 0 rpy=0 0.70 0; type revolute -> fixed
- joint fl_knee_joint: axis 0 -1 0 -> (none); limit lower=-2.792 upper=2.809 effort=76.4 velocity=22.4 -> (none); origin xyz=0 0.0984 -0.25 rpy=0 0 0 -> xyz=0 0.0984 -0.25 rpy=0 -1.40 0; type revolute -> fixed
- joint fr_hipx_joint: axis -1 0 0 -> (none); limit lower=-0.436 upper=0.611 effort=76.4 velocity=22.4 -> (none); type revolute -> fixed
- joint fr_hipy_joint: axis 0 -1 0 -> (none); limit lower=-2.583 upper=2.286 effort=76.4 velocity=22.4 -> (none); origin xyz=0 0 0 rpy=0 0 0 -> xyz=0 0 0 rpy=0 0.70 0; type revolute -> fixed
- joint fr_knee_joint: axis 0 -1 0 -> (none); limit lower=-2.792 upper=2.809 effort=76.4 velocity=22.4 -> (none); origin xyz=0 -0.0984 -0.25 rpy=0 0 0 -> xyz=0 -0.0984 -0.25 rpy=0 -1.40 0; type revolute -> fixed
- joint hl_hipx_joint: axis -1 0 0 -> (none); limit lower=-0.611 upper=0.436 effort=76.4 velocity=22.4 -> (none); type revolute -> fixed
- joint hl_hipy_joint: axis 0 -1 0 -> (none); limit lower=-2.286 upper=2.583 effort=76.4 velocity=22.4 -> (none); origin xyz=0 0 0 rpy=0 0 0 -> xyz=0 0 0 rpy=0 -0.70 0; type revolute -> fixed
- joint hl_knee_joint: axis 0 -1 0 -> (none); limit lower=-2.809 upper=2.792 effort=76.4 velocity=22.4 -> (none); origin xyz=0 0.0984 -0.25 rpy=0 0 0 -> xyz=0 0.0984 -0.25 rpy=0 1.40 0; type revolute -> fixed
- joint hr_hipx_joint: axis -1 0 0 -> (none); limit lower=-0.436 upper=0.611 effort=76.4 velocity=22.4 -> (none); type revolute -> fixed
- joint hr_hipy_joint: axis 0 -1 0 -> (none); limit lower=-2.286 upper=2.583 effort=76.4 velocity=22.4 -> (none); origin xyz=0 0 0 rpy=0 0 0 -> xyz=0 0 0 rpy=0 -0.70 0; type revolute -> fixed
- joint hr_knee_joint: axis 0 -1 0 -> (none); limit lower=-2.809 upper=2.792 effort=76.4 velocity=22.4 -> (none); origin xyz=0 -0.0984 -0.25 rpy=0 0 0 -> xyz=0 -0.0984 -0.25 rpy=0 1.40 0; type revolute -> fixed
